File: KiCad/BottomHeater.kicad_sch (KiCad schematic)
At the start: 13 parts, among them J1 Power In, J2 Load, Q1 BTA16-600B, U1 MOC3021M, U2 4N25

Commit message: work in progress
Parts:
- removed R5: R, symbol Device:R
- added D2: LED, LED_THT:LED_D3.0mm, symbol Device:LED
- added PS1: HLK-PM03, Converter_ACDC:Converter_ACDC_Hi-Link_HLK-PMxx, symbol Converter_ACDC:HLK-PM03
- added U3: MAX31855EASA, Package_SO:SOIC-8_3.9x4.9mm_P1.27mm, symbol Sensor_Temperature:MAX31855EASA
- R1: value R -> 1K
- R2: value R -> 58K
- R3: value R -> 10K; footprint (none) -> Resistor_SMD:R_0612_1632Metric_Pad1.18x3.40mm_HandSolder
- R4: value R -> 340
- R6: value R -> 470
Connections:
- net GND: now also A1.2 (GND), D2.1 (K), PS1.3 (-Vout), U3.1 (GND)
- net at J2.2 (Pin_2), Q1.1 (A1): no longer R3.1
- net at Q1.3 (G), U1.4: no longer R3.2
- net at R6.2: now also R4.2
- net at J1.1 (Pin_1), Q1.2 (A2), R1.1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: now also PS1.2 (AC/N)
- net at D1.4, J1.2 (Pin_2), J2.1 (Pin_1): now also PS1.1 (AC/L)
- net at A1.21 (VIN): now also PS1.4 (+Vout)
- net at R4.1: now also D2.2 (A); no longer U2.5
- new net: R3.1, U2.5
- no-connect marks 0 -> 1
Other:
- note added: "2.3v"
- note added: "DC 1.1v"
- note added: "pwm"
- note added: "vcc"
- note added: "zero-cross"
- moved on the sheet: A1, R6, U1

Commit message: board almost done
Parts:
- removed A1: Maple_Mini, Module:Maple_Mini, symbol MCU_Module:Maple_Mini
- added BT1: Battery_Cell, Battery:BatteryHolder_MYOUNG_BS-07-A1BJ001_CR2032, symbol Device:Battery_Cell
- added C1: 10 uF, Capacitor_SMD:C_0603_1608Metric, symbol Device:C
- added C2: C, Capacitor_SMD:C_0603_1608Metric, symbol Device:C
- added C3: C, Capacitor_THT:C_Radial_D5.0mm_H5.0mm_P2.00mm, symbol Device:C
- added H1, H2, H3, H4: MountingHole, MountingHole:MountingHole_2mm, symbol Mechanical:MountingHole
- added J3: Screw_Terminal_01x02, Connector_Phoenix_GMSTB:PhoenixContact_GMSTBVA_2,5_2-G-7,62_1x02_P7.62mm_Vertical, symbol Connector:Screw_Terminal_01x02
- added J4: Display 20x4, Connector_Molex:Molex_KK-254_AE-6410-05A_1x05_P2.54mm_Vertical, symbol Connector:Conn_01x04_Socket
- added J5: Encoder, Connector_Molex:Molex_KK-254_AE-6410-05A_1x05_P2.54mm_Vertical, symbol Connector:Conn_01x05_Socket
- added U5: YAAJ_BluePill_Part_Like, Library:YAAJ_BluePill_1, symbol STM32_Pills:YAAJ_BluePill_Part_Like
- J1, J2: footprint (none) -> TerminalBlock:TerminalBlock_MaiXu_MX126-5.0-02P_1x02_P5.00mm
- PS1: value HLK-PM03 -> HLK-PM05 (5v)
- R1: footprint Resistor_THT:R_Axial_DIN0516_L15.5mm_D5.0mm_P20.32mm_Horizontal -> Resistor_THT:R_Axial_DIN0309_L9.0mm_D3.2mm_P15.24mm_Horizontal
- R2: value 58K -> 60K 1w; footprint (none) -> Resistor_THT:R_Axial_DIN0309_L9.0mm_D3.2mm_P15.24mm_Horizontal
- R3: footprint Resistor_SMD:R_0612_1632Metric_Pad1.18x3.40mm_HandSolder -> Resistor_SMD:R_1206_3216Metric
- R4: footprint Resistor_SMD:R_1206_3216Metric_Pad1.30x1.75mm_HandSolder -> Resistor_SMD:R_1206_3216Metric
- R6: footprint (none) -> Resistor_SMD:R_1206_3216Metric
- U3: value MAX31855EASA -> MAX6675
Connections:
- net GND: now also U3.2 (T-), BT1.2 (-), C1.1, C2.2, C3.1, J3.1 (Pin_1), J4.1 (Pin_1), J5.1 (Pin_1), U5.19 (GND), U5.40 (GND)
- net at R4.2, R6.2: now also U5.36 (PB11)
- net at R3.1, U2.5: now also U5.35 (PB10)
- net at R3.2: now also U3.4 (V_CC), C2.1, J5.2 (Pin_2), U5.38 (3V3)
- net at J1.1 (Pin_1), Q1.2 (A2), R1.1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: now also PS1.1 (AC/L); no longer PS1.2 (AC/N)
- net at D1.4, J1.2 (Pin_2), J2.1 (Pin_1): now also PS1.2 (AC/N); no longer PS1.1 (AC/L)
- net at U3.3 (T+): now also J3.2 (Pin_2)
- net at U3.5 (SCK): now also U5.7 (PA10)
- net at U3.6 (~{CS}): now also U5.8 (PA11)
- net at U3.7 (SO): now also U5.9 (PA12)
- net at PS1.4 (+Vout): now also C1.2, C3.2, J4.2 (Pin_2), U5.18 (5V)
- new net: J4.3 (Pin_3), U5.15 (PB7)
- new net: J4.4 (Pin_4), U5.14 (PB6)
- new net: J5.3 (Pin_3), U5.6 (PA9)
- new net: J5.4 (Pin_4), U5.5 (PA8)
- new net: J5.5 (Pin_5), U5.4 (PB15)
- new net: BT1.1 (+), U5.21 (VBat)
Other:
- moved on the sheet: D1, D2, J1, J2, PS1, Q1, R1, R2, R3, R4, R6, U1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
